File: hardware/rpi-pico-debugger-shoe/rpi-pico-debugger-shoe.kicad_pcb (KiCad board)
At the start: 2 copper layers, 43 parts, among them J1 10118193-0001LF, J2 Conn_01x02, J3 Conn_01x03, J4 Conn_01x18, J5 Conn_01x20, J6 Conn_01x03, J7 Conn_01x03, J8 Conn_01x02, SW1 PTS810_SJK_250_SMTR_LFS, U1 RP2040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

Commit message: Did done some layouts
Parts:
- added FID1: Fiducial, Fiducial:Fiducial_1mm_Mask2mm, F.Cu at (135.1, 93.6)
- added FID2: Fiducial, Fiducial:Fiducial_1mm_Mask2mm, F.Cu at (143.2, 121.3)
- added H1: MountingHole, MountingHole:MountingHole_2.1mm, F.Cu at (131.8, 78.0)
- added H2: MountingHole, MountingHole:MountingHole_2.1mm, F.Cu at (143.2, 78.0)
- added H3: MountingHole, MountingHole:MountingHole_2.1mm, F.Cu at (131.8, 125.0)
- added H4: MountingHole, MountingHole:MountingHole_2.1mm, F.Cu at (143.2, 125.0)
- JP1, JP2, JP3: moved to B.Cu
- moved J6 68.6 mm to (135.0, 125.4), turned to 90 degrees
- moved J7 50.6 mm to (135.0, 129.2), turned to 90 degrees
- moved Y1 47.3 mm to (137.5, 113.5)
- moved LED1 45.9 mm to (142.6, 118.5), turned to 180 degrees
- moved J2 45.2 mm to (136.2, 120.3), turned to 90 degrees
- moved U1 44.6 mm to (137.5, 104.5)
- moved J3 42.0 mm to (135.0, 122.9), turned to 90 degrees
- moved J8 28.0 mm to (128.6, 77.4)
- moved C13 27.8 mm to (135.8, 116.8)
- moved C11 27.6 mm to (142.6, 110.4)
- moved C15 25.7 mm to (139.2, 116.8), turned to 180 degrees
- moved JP3 23.4 mm to (142.0, 82.5), turned to 180 degrees
- moved C1 23.4 mm to (134.5, 97.5), turned to 90 degrees
- moved C6 22.9 mm to (139.5, 85.5), turned to 90 degrees
- moved C3 22.8 mm to (132.0, 106.3), turned to 270 degrees
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Routing:
- net +3V3: track 0.00 -> 75.0 mm, vias 0 -> 2
- net /TARGET_TX: track 0.00 -> 30.5 mm, vias 0 -> 1
- net /TARGET_RX: track 0.00 -> 27.0 mm, vias 0 -> 1
- net /QSPI_SD0: track 0.00 -> 22.4 mm, vias 0 -> 2
- net /QSPI_SD3: track 0.00 -> 19.7 mm, vias 0 -> 2
- net /QSPI_SCK: track 0.00 -> 19.2 mm, vias 0 -> 2
- net /USB_P: track 0.00 -> 16.0 mm
- net /USB_N: track 0.00 -> 16.0 mm
- net /QSPI_CS: track 0.00 -> 16.0 mm, vias 0 -> 2
- net /QSPI_SD1: track 0.00 -> 14.8 mm, vias 0 -> 2
- net /QSPI_SD2: track 0.00 -> 13.9 mm, vias 0 -> 2
- net /VSYS: track 0.00 -> 9.56 mm, vias 0 -> 1
- net Net-(J8-Pad1): track 0.00 -> 5.98 mm
- net Net-(J8-Pad2): track 0.00 -> 5.94 mm
- net Net-(J5-Pad2): track 0.00 -> 4.81 mm
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Other:
- board outline added: 21 x 54.5 mm
- net class Default: clearance 0.2 -> 0.22; trace_width 0.25 -> 0.18; via_dia 0.8 -> 0.508; via_drill 0.4 -> 0.254
- net class Power added: clearance 0.22, trace_width 0.3, via_dia 0.508, via_drill 0.254
- net class USB Data added: clearance 0.22, trace_width 0.18, via_dia 0.508, via_drill 0.254
- rule pad_to_mask_clearance: 0 -> 0.0508
- rule trace_clearance: 0.2 -> 0.22
- rule trace_min: 0.2 -> 0.1524
- rule via_min_drill: 0.3 -> 0.254
- rule via_min_size: 0.4 -> 0.508

Commit message: Finished layout for v01
Parts:
- J1: footprint 10118193-0001LF:FCI_10118193-0001LF -> 10118193-0001LF:FCI_10118193-0001LF_no-slot
- J2, J8: footprint Connector_PinHeader_2.54mm:PinHeader_1x02_P2.54mm_Vertical -> custom:PinHeader_1x02_P2.54mm_Vertical_no-silk
- J3, J6, J7: footprint Connector_PinHeader_2.54mm:PinHeader_1x03_P2.54mm_Vertical -> custom:PinHeader_1x03_P2.54mm_Vertical_no-silk
- J4: footprint Connector_PinHeader_2.54mm:PinHeader_1x18_P2.54mm_Vertical -> custom:PinHeader_1x18_P2.54mm_Vertical_no-silk
- J5: footprint Connector_PinHeader_2.54mm:PinHeader_1x20_P2.54mm_Vertical -> custom:PinHeader_1x20_P2.54mm_Vertical_no-silk
- moved C1 0.90 mm to (135.2, 97.0)
- moved C10 0.90 mm to (141.2, 97.0)
- moved C12 0.90 mm to (139.8, 97.0)
- moved C9 0.90 mm to (133.8, 97.0)
- moved R4 0.90 mm to (136.8, 97.0)
- moved R5 0.90 mm to (138.2, 97.0)
- moved SW1 0.80 mm to (141.6, 92.5), turned to 180 degrees
Connections:
- J5 pad 8: Net-(J5-Pad8) -> GND
Routing:
- net +3V3: track 75.0 -> 126.0 mm
- net /TARGET_SWDIO: track 0.00 -> 37.3 mm, vias 0 -> 1
- net /USB_BOOT: track 0.00 -> 37.1 mm, vias 0 -> 3
- net /TARGET_SWCLK: track 0.00 -> 35.1 mm, vias 0 -> 1
- net /+1.1V: track 0.00 -> 25.8 mm, vias 0 -> 2
- net /SWCLK: track 0.00 -> 24.5 mm, vias 0 -> 1
- net /SWDIO: track 0.00 -> 21.0 mm, vias 0 -> 1
- net /RUN: track 0.00 -> 20.6 mm, vias 0 -> 2
- net /GPIO25: track 0.00 -> 15.4 mm, vias 0 -> 2
- net /XIN: track 0.00 -> 15.1 mm
- net Net-(C15-Pad1): track 0.00 -> 9.23 mm
- net GND: track 0.00 -> 7.47 mm, vias 0 -> 47
- net /XOUT: track 0.00 -> 5.91 mm
- net /QSPI_CS: track 16.0 -> 19.6 mm
- net /QSPI_SCK: track 19.2 -> 22.1 mm
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- added copper zone on B.Cu, net GND
- added copper zone on F.Cu, net GND
Other:
- board size 21 x 54.5 mm -> 25.4 x 54.5 mm
- rule pad_to_mask_clearance: 0.0508 -> 0
- board text added: "10"
- board text added: "11"
- board text added: "12"
- board text added: "13"
- board text added: "14"
- board text added: "15"
- board text added: "16"
- board text added: "17"
- board text added: "18"
- board text added: "19"
- board text added: "2"
- board text added: "20"
- board text added: "21"
- board text added: "22"
- board text added: "26"
- board text added: "27"
- board text added: "28"
- board text added: "3"
- board text added: "3V3"
- board text added: "4"
- board text added: "5"
- board text added: "6"
- board text added: "7"
- board text added: "8"
- board text added: "9"
- board text added: "AREF"
- board text added: "BTSEL"
- board text added: "CLK"
- board text added: "DIO"
- board text added: "EN"
- board text added: "GND"
- board text added: "RESET"
- board text added: "RPi Pico Debugger Shoe"
- board text added: "RUN"
- board text added: "SHOE SWD"
- board text added: "TGT_RX"
- board text added: "TGT_TX"
- board text added: "VBUS"
- board text added: "VSYS"
- board text added: "v01"
